File: project/project.kicad_sch (KiCad schematic)
At the start: 41 parts, among them J101 BUS, J102 rs485, J103 qwiic, J104 FFC, J105 Bot, J106 FFC, J107 Top, J108 Mid, J109 Mid, J110 USB_C_Receptacle_USB2.0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

Commit message: fix PSU FB and tmp102 pinout
Parts:
- U101, U104: footprint Package_TO_SOT_SMD:SOT-563 -> -local:SOT-563; symbol Sensor_Temperature:TMP101 -> Sensor_Temperature:TMP102xxDRL
Connections:
- net 3V3: now also U104.5 (V+); no longer U101.4 (V+), U104.4 (V+)
- net GND: now also U104.4 (ADD0); no longer U104.5 (ADD0)
- net SDA: now also U101.4 (ADD0)
Other:
- note added: "I2C: 0x48"
- note added: "I2C: 0x4A"
- note removed: "I2C addr: 0x48"
- note removed: "I2C addr: 0x4A"
Changed lines of the file:
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@@
     (effects (font (size 2 2)) (justify right bottom))
   )
-  (text "I2C\naddr:\n0x48" (at 215.9 40.64 180)
+  (text "I2C:\n0x48" (at 215.9 40.64 180)
     (effects (font (size 2 2)) (justify right bottom))
   )
@@
     (effects (font (size 5 5) (thickness 0.6) bold) (justify left bottom))
   )
-  (text "I2C addr:\n0x4A" (at 67.31 40.64 180)
+  (text "I2C:\n0x4A" (at 67.31 40.64 180)
     (effects (font (size 2 2)) (justify right bottom))
   )
@@
     )
   )
-  (global_label "3V3" (shape input) (at 68.58 33.02 180) (fields_autoplaced)
-    (effects (font (size 1.27 1.27)) (justify right))
-    (property "Intersheet References" "${INTERSHEET_REFS}" (id 0) (at 62.6593 32.9406 0)
-      (effects (font (size 1.27 1.27)) (justify right) hide)
-    )
-  )
   (global_label "M_USR_LED" (shape input) (at 275.59 88.9 90) (fields_autoplaced)
     (effects (font (size 1.27 1.27)) (justify left))
@@
     (property "Intersheet References" "${INTERSHEET_REFS}" (id 0) (at 155.4179 49.4506 0)
       (effects (font (size 1.27 1.27)) (justify left) hide)
+    )
+  )
+  (global_label "SDA" (shape input) (at 68.58 33.02 180) (fields_autoplaced)
+    (effects (font (size 1.27 1.27)) (justify right))
+    (property "Intersheet References" "${INTERSHEET_REFS}" (id 0) (at 62.5988 32.9406 0)
+      (effects (font (size 1.27 1.27)) (justify right) hide)
     )
   )
@@
     (pin "2")
   )
-  (symbol (lib_id "Sensor_Temperature:TMP101") (at 227.33 31.75 0) (unit 1)
+  (symbol (lib_id "Sensor_Temperature:TMP102xxDRL") (at 227.33 31.75 0) (unit 1)
     (in_bom yes) (on_board yes)
     (property "Reference" "U104" (id 0) (at 220.98 22.86 0))
-    (property "Value" "TMP102" (id 1) (at 222.25 40.64 0))
-    (property "Footprint" "Package_TO_SOT_SMD:SOT-563" (id 2) (at 228.6 40.64 0)
-      (effects (font (size 1.27 1.27)) (justify left) hide)
-    )
-    (property "Datasheet" "https://www.lcsc.com/datasheet/C99269.pdf" (id 3) (at 228.6 43.18 0)
+    (property "Value" "TMP102" (id 1) (at 232.41 40.64 0))
+    (property "Footprint" "-local:SOT-563" (id 2) (at 228.6 40.64 0)
+      (effects (font (size 1.27 1.27)) (justify left) hide)
+    )
+    (property "Datasheet" "https://www.ti.com/lit/ds/symlink/tmp102.pdf" (id 3) (at 228.6 43.18 0)
       (effects (font (size 1.27 1.27)) (justify left) hide)
     )
@@
     (pin "MP")
   )
-  (symbol (lib_id "Sensor_Temperature:TMP101") (at 78.74 31.75 0) (unit 1)
+  (symbol (lib_id "Sensor_Temperature:TMP102xxDRL") (at 78.74 31.75 0) (unit 1)
     (in_bom yes) (on_board yes)
     (property "Reference" "U101" (id 0) (at 72.39 22.86 0))
-    (property "Value" "TMP102" (id 1) (at 73.66 40.64 0))
-    (property "Footprint" "Package_TO_SOT_SMD:SOT-563" (id 2) (at 80.01 40.64 0)
-      (effects (font (size 1.27 1.27)) (justify left) hide)
-    )
-    (property "Datasheet" "https://www.lcsc.com/datasheet/C99269.pdf" (id 3) (at 80.01 43.18 0)
+    (property "Value" "TMP102" (id 1) (at 83.82 40.64 0))
+    (property "Footprint" "-local:SOT-563" (id 2) (at 80.01 40.64 0)
+      (effects (font (size 1.27 1.27)) (justify left) hide)
+    )
+    (property "Datasheet" "https://www.ti.com/lit/ds/symlink/tmp102.pdf" (id 3) (at 80.01 43.18 0)
       (effects (font (size 1.27 1.27)) (justify left) hide)
     )
@@
     )
     (path "/a8beda3e-8147-457c-a4ed-0b9d9627967c"
-      (reference "U101") (unit 1) (value "TMP102") (footprint "Package_TO_SOT_SMD:SOT-563")
+      (reference "U101") (unit 1) (value "TMP102") (footprint "-local:SOT-563")
     )
     (path "/e6411339-b124-42ec-a9a0-8664f864a926"
@@
     )
     (path "/55cbd1b5-ecb1-4b1b-9a94-3461217e0d3f"
-      (reference "U104") (unit 1) (value "TMP102") (footprint "Package_TO_SOT_SMD:SOT-563")
+      (reference "U104") (unit 1) (value "TMP102") (footprint "-local:SOT-563")
     )
     (path "/33ae409b-a770-4e46-a271-f5b63686e12b"
