File: project/project.kicad_pcb (KiCad board)
At the start: 4 copper layers, 64.5 x 86 mm, 186 parts, among them J101 BUS, J102 rs485, J103 qwiic, J104 FFC, J105 Bot, J106 FFC, J107 Top, J108 Mid, J109 Mid, J110 USB_C_Receptacle_USB2.0, J111 BUS, J201 5V, J202 24V, J203 3V3, J401 RJ45_Shielded, SW101 15mm, SW102 15mm, U101 TMP102, U102 24C02S, U103 USBLC6-2SC6, U104 TMP102, U105 INA226, U201 DP9700AT-24, U202 ME3121AM6G, U203 JTD6206-3.3V, U301 esp32-C3FH4X, U401 W5500, U501 XL1050, U601 MAX13487E, Y301 40MHz, Y401 25MHz

Commit message: CAN resistors, power wires and version bump
* fixing CAN level shifting resistors
* exposing more copper for power wires between boards
* bumping up version
Parts:
- removed kibuzzard-69A9CD9B: G***, kibuzzard-69A9CD9B
- removed kibuzzard-69AFDE57 (x2): G***, kibuzzard-69AFDE57
- added R507: 3k, Resistor_SMD:R_0402_1005Metric_Pad0.72x0.64mm_HandSolder, F.Cu at (199.7, 61.5)
- added kibuzzard-6A7A3E96: G***, kibuzzard-6A7A3E96, F.Cu at (191.6, 54.2)
- added kibuzzard-6A7A3EB1: G***, kibuzzard-6A7A3EB1, B.Cu at (151.4, 50.4)
- added kibuzzard-6A7A3F37: G***, kibuzzard-6A7A3F37, F.Cu at (163.5, 81.5)
- R501: value 4k7 -> 1k5
- moved C303 2.92 mm to (195.7, 58.7), turned to 180 degrees
- moved D501 1.50 mm to (195.6, 55.5)
- moved D502 1.50 mm to (193.6, 55.5)
- moved R502 1.50 mm to (194.5, 52.0)
- renumbered U301 to locked
Routing:
- net GND: track 59.6 -> 61.8 mm, vias 623 -> 622
- net CAN_LED: track 3.93 -> 2.43 mm
- net /uC/XTAL_N: track 4.36 -> 5.67 mm
- net /CAN_TX: track 10.7 -> 9.74 mm
- net /CAN/CAN_RX5: track 13.8 -> 13.1 mm
Other:
- board text added: "WC GwPoeAt"
