File: project/project.kicad_pcb (KiCad board)
At the start: 4 copper layers, 64.5 x 86 mm, 187 parts, among them J101 BUS, J102 rs485, J103 qwiic, J104 FFC, J105 Bot, J106 FFC, J107 Top, J108 Mid, J109 Mid, J110 USB_C_Receptacle_USB2.0, J111 BUS, J201 5V, J202 24V, J203 3V3, J401 RJ45_Shielded, SW101 15mm, SW102 15mm, U101 TMP102, U102 24C02S, U103 USBLC6-2SC6, U104 TMP102, U105 INA226, U201 DP9700AT-24, U202 ME3121AM6G, U203 JTD6206-3.3V, U401 W5500, U501 XL1050, U601 MAX13487E, Y301 40MHz, Y401 25MHz

Commit message: adding fuse to power monitor to prevent reverse polarity damage
Parts:
- added C105: 100n, Capacitor_SMD:C_0402_1005Metric_Pad0.74x0.62mm_HandSolder, F.Cu at (162.3, 115.6)
- added F101: 10mA, Fuse:Fuse_0805_2012Metric_Pad1.15x1.40mm_HandSolder, F.Cu at (161.5, 112.0)
- added F102: 10mA, Fuse:Fuse_0805_2012Metric_Pad1.15x1.40mm_HandSolder, F.Cu at (163.5, 112.0)
- moved U105 3.26 mm to (166.0, 115.6), turned to 180 degrees
- moved C104 1.80 mm to (166.0, 113.3), turned to 0 degrees
- moved C103 0.71 mm to (166.5, 111.0), turned to 180 degrees
- moved R104 0.30 mm to (141.3, 97.5)
- moved R105 0.30 mm to (141.3, 100.0)
Connections:
- U105 pad 10: VOUT -> /ISNS_P
- U105 pad 8: VOUT -> /ISNS_P
- U105 pad 9: M_VCC -> /ISNS_N
Routing:
- net /ISNS_P: track 0.00 -> 7.41 mm
- net /ISNS_N: track 0.00 -> 5.02 mm
- net M_SCL: track 48.9 -> 44.8 mm
- net M_SDA: track 53.0 -> 49.2 mm
- net VOUT: track 10.8 -> 7.56 mm
- net 3V3: track 310.9 -> 309.0 mm, vias 20 -> 21
- net GND: track 61.8 -> 61.9 mm, vias 622 -> 618
Other:
- board text added: "CANL CANH GND 24V"
